Commit message: base corrected urdf

File: ManualPhase1/Ros/roboticarm_description/urdf/roboticarm.xacro (robot description, xacro)
@@ -6,7 +6,7 @@
 <link name="base_link">
   <inertial>
-    <origin xyz="-6.126236204605508e-05 0.0 0.3559553216998673" rpy="0 0 0"/>
-    <mass value="549.7939786248483"/>
-    <inertia ixx="27.124843" iyy="27.12698" izz="8.618743" ixy="0.0" iyz="0.0" ixz="0.012393"/>
+    <origin xyz="0.07170147470861574 0.0724672454182439 0.3244590303819093" rpy="0 0 0"/>
+    <mass value="555.7346839951744"/>
+    <inertia ixx="27.918915" iyy="27.919482" izz="8.711404" ixy="-0.000347" iyz="0.003477" ixz="0.00733"/>
   </inertial>
   <visual>
@@ -26,10 +26,10 @@
 <link name="waist_1">
   <inertial>
-    <origin xyz="-4.163336342344337e-16 0.0009104427321459631 0.015903844796416045" rpy="0 0 0"/>
+    <origin xyz="-4.5394164495393685e-07 0.000910466670597028 0.0159037153558238" rpy="0 0 0"/>
     <mass value="2.5376552135525894"/>
     <inertia ixx="0.006217" iyy="0.006015" izz="0.010077" ixy="0.0" iyz="-5e-05" ixz="0.0"/>
   </inertial>
   <visual>
-    <origin xyz="0.0635 -0.0 -0.7366" rpy="0 0 0"/>
+    <origin xyz="-0.034565 -0.054849 -0.708914" rpy="0 0 0"/>
     <geometry>
       <mesh filename="file://$(find roboticarm_description)/meshes/waist_1.stl" scale="0.001 0.001 0.001"/>
@@ -38,5 +38,5 @@
   </visual>
   <collision>
-    <origin xyz="0.0635 -0.0 -0.7366" rpy="0 0 0"/>
+    <origin xyz="-0.034565 -0.054849 -0.708914" rpy="0 0 0"/>
     <geometry>
       <mesh filename="file://$(find roboticarm_description)/meshes/waist_1.stl" scale="0.001 0.001 0.001"/>
@@ -46,10 +46,10 @@
 <link name="shoulder_1">
   <inertial>
-    <origin xyz="9.71445146547012e-17 -0.03584553168598965 0.1906430525761622" rpy="0 0 0"/>
+    <origin xyz="-4.5394164471801446e-07 -0.035845507747538544 0.19064392313557188" rpy="0 0 0"/>
     <mass value="8.062761032384062"/>
     <inertia ixx="0.067114" iyy="0.067471" izz="0.005059" ixy="0.0" iyz="-0.0003" ixz="-0.0"/>
   </inertial>
   <visual>
-    <origin xyz="0.0635 -0.03777 -0.788518" rpy="0 0 0"/>
+    <origin xyz="-0.034565 -0.092619 -0.760831" rpy="0 0 0"/>
     <geometry>
       <mesh filename="file://$(find roboticarm_description)/meshes/shoulder_1.stl" scale="0.001 0.001 0.001"/>
@@ -58,5 +58,5 @@
   </visual>
   <collision>
-    <origin xyz="0.0635 -0.03777 -0.788518" rpy="0 0 0"/>
+    <origin xyz="-0.034565 -0.092619 -0.760831" rpy="0 0 0"/>
     <geometry>
       <mesh filename="file://$(find roboticarm_description)/meshes/shoulder_1.stl" scale="0.001 0.001 0.001"/>
@@ -66,10 +66,10 @@
 <link name="elbow_1">
   <inertial>
-    <origin xyz="-7.231520749681475e-05 -0.03320584879402316 0.15559840828012983" rpy="0 0 0"/>
+    <origin xyz="-7.27691491417895e-05 -0.03320582485557203 0.1555982788395438" rpy="0 0 0"/>
     <mass value="7.521482396242973"/>
     <inertia ixx="0.04938" iyy="0.04967" izz="0.004753" ixy="1e-06" iyz="0.000784" ixz="-8.9e-05"/>
   </inertial>
   <visual>
-    <origin xyz="0.0635 -0.03363 -1.115644" rpy="0 0 0"/>
+    <origin xyz="-0.034565 -0.088479 -1.087958" rpy="0 0 0"/>
     <geometry>
       <mesh filename="file://$(find roboticarm_description)/meshes/elbow_1.stl" scale="0.001 0.001 0.001"/>
@@ -78,5 +78,5 @@
   </visual>
   <collision>
-    <origin xyz="0.0635 -0.03363 -1.115644" rpy="0 0 0"/>
+    <origin xyz="-0.034565 -0.088479 -1.087958" rpy="0 0 0"/>
     <geometry>
       <mesh filename="file://$(find roboticarm_description)/meshes/elbow_1.stl" scale="0.001 0.001 0.001"/>
@@ -86,10 +86,10 @@
 <link name="w_a_1">
   <inertial>
-    <origin xyz="9.409140133698202e-15 -0.00013480940033086986 0.023018024103573786" rpy="0 0 0"/>
+    <origin xyz="-4.539416358084747e-07 -0.0001347854618797828 0.023017894662987537" rpy="0 0 0"/>
     <mass value="0.32955278928588533"/>
     <inertia ixx="0.000115" iyy="7.4e-05" izz="6.3e-05" ixy="0.0" iyz="1e-06" ixz="0.0"/>
   </inertial>
   <visual>
-    <origin xyz="0.064008 0.000838 -1.418539" rpy="0 0 0"/>
+    <origin xyz="-0.034057 -0.054011 -1.390853" rpy="0 0 0"/>
     <geometry>
       <mesh filename="file://$(find roboticarm_description)/meshes/w_a_1.stl" scale="0.001 0.001 0.001"/>
@@ -98,5 +98,5 @@
   </visual>
   <collision>
-    <origin xyz="0.064008 0.000838 -1.418539" rpy="0 0 0"/>
+    <origin xyz="-0.034057 -0.054011 -1.390853" rpy="0 0 0"/>
     <geometry>
       <mesh filename="file://$(find roboticarm_description)/meshes/w_a_1.stl" scale="0.001 0.001 0.001"/>
@@ -106,10 +106,10 @@
 <link name="w_b_1">
   <inertial>
-    <origin xyz="6.022959908591474e-15 -0.023736499999999848 0.011335623939424444" rpy="0 0 0"/>
+    <origin xyz="-4.5394163915302155e-07 -0.023736476061548904 0.011335494498837306" rpy="0 0 0"/>
     <mass value="0.03411828668710707"/>
     <inertia ixx="2.4e-05" iyy="6e-06" izz="2e-05" ixy="0.0" iyz="0.0" ixz="-0.0"/>
   </inertial>
   <visual>
-    <origin xyz="0.064008 -0.021768 -1.455547" rpy="0 0 0"/>
+    <origin xyz="-0.034057 -0.076617 -1.427861" rpy="0 0 0"/>
     <geometry>
       <mesh filename="file://$(find roboticarm_description)/meshes/w_b_1.stl" scale="0.001 0.001 0.001"/>
@@ -118,5 +118,5 @@
   </visual>
   <collision>
-    <origin xyz="0.064008 -0.021768 -1.455547" rpy="0 0 0"/>
+    <origin xyz="-0.034057 -0.076617 -1.427861" rpy="0 0 0"/>
     <geometry>
       <mesh filename="file://$(find roboticarm_description)/meshes/w_b_1.stl" scale="0.001 0.001 0.001"/>
@@ -126,10 +126,10 @@
 <link name="w_c_1">
   <inertial>
-    <origin xyz="-0.003951491072912233 -0.027299401705366138 0.06838528705274549" rpy="0 0 0"/>
+    <origin xyz="-0.003951945014557701 -0.027299377766914802 0.06838515761215969" rpy="0 0 0"/>
     <mass value="0.6216016037280759"/>
     <inertia ixx="0.001485" iyy="0.001254" izz="0.000602" ixy="6.7e-05" iyz="0.000585" ixz="-0.000116"/>
   </inertial>
   <visual>
-    <origin xyz="0.064008 0.001968 -1.482547" rpy="0 0 0"/>
+    <origin xyz="-0.034057 -0.052881 -1.454861" rpy="0 0 0"/>
     <geometry>
       <mesh filename="file://$(find roboticarm_description)/meshes/w_c_1.stl" scale="0.001 0.001 0.001"/>
@@ -138,5 +138,5 @@
   </visual>
   <collision>
-    <origin xyz="0.064008 0.001968 -1.482547" rpy="0 0 0"/>
+    <origin xyz="-0.034057 -0.052881 -1.454861" rpy="0 0 0"/>
     <geometry>
       <mesh filename="file://$(find roboticarm_description)/meshes/w_c_1.stl" scale="0.001 0.001 0.001"/>
@@ -146,10 +146,10 @@
 <link name="gripper_1">
   <inertial>
-    <origin xyz="-1.0010543181615539e-06 -0.004373051617807485 0.05098724133949806" rpy="0 0 0"/>
+    <origin xyz="-1.4549959634693743e-06 -0.004374027679356865 0.05098711189891225" rpy="0 0 0"/>
     <mass value="0.7040814534189734"/>
     <inertia ixx="0.00099" iyy="0.000924" izz="0.000643" ixy="-0.0" iyz="9.8e-05" ixz="-0.0"/>
   </inertial>
   <visual>
-    <origin xyz="0.064008 0.001969 -1.569747" rpy="0 0 0"/>
+    <origin xyz="-0.034057 -0.052881 -1.542061" rpy="0 0 0"/>
     <geometry>
       <mesh filename="file://$(find roboticarm_description)/meshes/gripper_1.stl" scale="0.001 0.001 0.001"/>
@@ -158,5 +158,5 @@
   </visual>
   <collision>
-    <origin xyz="0.064008 0.001969 -1.569747" rpy="0 0 0"/>
+    <origin xyz="-0.034057 -0.052881 -1.542061" rpy="0 0 0"/>
     <geometry>
       <mesh filename="file://$(find roboticarm_description)/meshes/gripper_1.stl" scale="0.001 0.001 0.001"/>
@@ -165,11 +165,11 @@
 </link>
 <joint name="Revolute 11" type="continuous">
-  <origin xyz="-0.0635 0.0 0.7366" rpy="0 0 0"/>
+  <origin xyz="0.034565 0.054849 0.708914" rpy="0 0 0"/>
   <parent link="base_link"/>
   <child link="waist_1"/>
-  <axis xyz="0.0 0.0 -1.0"/>
+  <axis xyz="0.0 -0.0 -1.0"/>
 </joint>
 <joint name="Revolute 12" type="continuous">
-  <origin xyz="0.0 0.03777 0.051918" rpy="0 0 0"/>
+  <origin xyz="0.0 0.03777 0.051917" rpy="0 0 0"/>
   <parent link="waist_1"/>
   <child link="shoulder_1"/>
@@ -177,8 +177,8 @@
 </joint>
 <joint name="Revolute 13" type="continuous">
-  <origin xyz="0.0 -0.00414 0.327126" rpy="0 0 0"/>
+  <origin xyz="0.0 -0.00414 0.327127" rpy="0 0 0"/>
   <parent link="shoulder_1"/>
   <child link="elbow_1"/>
-  <axis xyz="0.0 1.0 0.0"/>
+  <axis xyz="0.0 1.0 -0.0"/>
 </joint>
 <joint name="Revolute 18" type="continuous">
@@ -186,5 +186,5 @@
   <parent link="elbow_1"/>
   <child link="w_a_1"/>
-  <axis xyz="0.0 0.0 1.0"/>
+  <axis xyz="-0.0 0.0 1.0"/>
 </joint>
 <joint name="Revolute 19" type="continuous">
@@ -192,5 +192,5 @@
   <parent link="w_a_1"/>
   <child link="w_b_1"/>
-  <axis xyz="0.0 1.0 0.0"/>
+  <axis xyz="0.0 1.0 -0.0"/>
 </joint>
 <joint name="Revolute 20" type="continuous">
@@ -201,5 +201,5 @@
 </joint>
 <joint name="Rigid 21" type="fixed">
-  <origin xyz="0.0 -1e-06 0.0872" rpy="0 0 0"/>
+  <origin xyz="0.0 0.0 0.0872" rpy="0 0 0"/>
   <parent link="w_c_1"/>
   <child link="gripper_1"/>
