Commit message: pipeline done, web-->ik-->bridge

File: ManualPhase1/ROBO_ws/src/roboticarm_description/urdf/roboticarm.xacro (robot description, xacro)
@@ -151,5 +151,5 @@
   </inertial>
   <visual>
-    <origin xyz="0.160761 -0.364037 -0.437465" rpy="0 0 0"/>
+    <origin xyz="-0.160761 -0.364037 0.437465" rpy="0 3.14159265 0"/>
     <geometry>
       <mesh filename="file://$(find roboticarm_description)/meshes/gripper_1.stl" scale="0.001 0.001 0.001"/>
@@ -158,5 +158,5 @@
   </visual>
   <collision>
-    <origin xyz="0.160761 -0.364037 -0.437465" rpy="0 0 0"/>
+    <origin xyz="-0.160761 -0.364037 0.437465" rpy="0 3.14159265 0"/>
     <geometry>
       <mesh filename="file://$(find roboticarm_description)/meshes/gripper_1.stl" scale="0.001 0.001 0.001"/>
@@ -224,5 +224,5 @@
 </joint>
 <joint name="Rigid 49" type="fixed">
-  <origin xyz="-0.0872 0.0 0.0" rpy="0 0 0"/>
+  <origin xyz="-0.0872 0.0 0.0" rpy="0 3.14159265 0"/>
   <parent link="w_c_1"/>
   <child link="gripper_1"/>
